File: v3-tb.sch (EAGLE design)
At the start: 47 parts, among them J1 MPU_SPI, J10 HRDAC, J11 AMPS, J12 CDC_PC, J13 GROUND, J2 MCU_SPI, J3 MPU_I2C, J4 MPU_ETC, J5 MCU_ETC, J7 POWER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

Commit message: Add board
Parts:
- J13: value GROUND -> GND
- J7: value POWER -> (none)
Connections:
- removed net MISO: J1.1, J2.1, U4.MISO_PG1, U5.MISO, U7.H_SDA/MISO/TX
- removed net MOSI: J1.2, J2.2, U4.MOSI_SDA, U5.MOSI, U7.H_SA0/MOSI
- removed net SCK: J1.3, J2.3, U4.SCK_SCL, U5.SCLK, U7.H_SCL/SCLK/RX
- removed net SCL: J3.1, U6.SCL
- removed net SDA: J3.2, U6.SDA
- new net MCU_MISO: J2.2, U4.MISO_PG1
- new net MCU_MOSI: J2.1, U4.MOSI_SDA
- new net MCU_SCK: J2.3, U4.SCK_SCL
- new net MPU_MISO: J1.2, U5.MISO, U7.H_SDA/MISO/TX
- new net MPU_MOSI: J1.1, U5.MOSI, U7.H_SA0/MOSI
- new net MPU_SCK: J1.3, U5.SCLK, U7.H_SCL/SCLK/RX
- new net MPU_SCL: J3.2, U6.SCL
- new net MPU_SDA: J3.1, U6.SDA
- net CDC_PC0: now also J12.3; no longer J12.1
- net CDC_PC1: now also J12.4; no longer J12.2
- net CDC_PC2: now also J12.5; no longer J12.3
- net CDC_PC3: now also J12.6; no longer J12.4
- net CDC_PC4: now also J12.1; no longer J12.5
- net CDC_PC5: now also J12.2; no longer J12.6
